File: board/board.kicad_sch (KiCad schematic)
At the start: 1 part

Commit message: initial
Parts:
- added J1: 001_I2C, on_edge:on_edge_2x05_device, symbol put_on_edge:001_I2C
- added J2: 008_USB, on_edge:on_edge_2x05_device, symbol put_on_edge:008_USB
- added TP1: TestPoint, TestPoint:TestPoint_Loop_D3.80mm_Drill2.8mm, symbol Connector:TestPoint
Connections:
- net GND: now also J1.1 (GND), J2.1 (GND)
- new net charger/Bat+: TP1.1
- new net charger/SCL: J1.4 (SCL)
- new net charger/SDA: J1.2 (SDA)
- new net charger/V3.3: J1.9 (3.3V)
- new net charger/Vin: J2.10 (5V)
Other:
- sheet implementation renamed charger
- sheet charger: file implementation.kicad_sch -> charger.kicad_sch
- sheet charger ports: added Bat+, SCL, SDA, V3.3, Vin; removed none
- note removed: "Input connectors go here"
- note removed: "Output connectors go here"
